Commit message: Updated camera RPY to use PI instead of pi
I found when compiling this on my own system that compilation failed with the following error - "xacro.XacroException: Property wasn't defined: u'pi'". I found that this file defined PI but used pi. Changing this to PI on my system fixed it so I thought you might appreciate the same.

File: rrbot_description/urdf/rrbot.xacro (robot description, xacro)
@@ -165,5 +165,5 @@
     <!-- these values have to be these values otherwise the gazebo camera image
         won't be aligned properly with the frame it is supposedly originating from -->
-    <origin xyz="0 0 0" rpy="${-pi/2} 0 ${-pi/2}"/>
+    <origin xyz="0 0 0" rpy="${-PI/2} 0 ${-PI/2}"/>
     <parent link="camera_link"/>
     <child link="camera_link_optical"/>
